Commit message: adding updated arduino code

File: src/prototype/urdf/joint_macros.xacro (robot description, xacro)
@@ -5,5 +5,5 @@
    <!--===============xacro for continuous joints=========================-->
     <xacro:macro name="joint_wheel" params="name origin parent child">
-        <joint name="${name}" type="fixed">
+        <joint name="${name}" type="continuous">
             <origin xyz="${origin}" rpy="0.0 0.0 0.0"/>
             <parent link="${parent}"/>

File: src/prototype/urdf/sattava_main.xacro (robot description, xacro)
@@ -6,5 +6,5 @@
     <xacro:include filename="joint_macros.xacro"/>
     <xacro:include filename="wheel.xacro"/>
-    <xacro:include filename="hardware_interface"/>
+    <xacro:include filename="hardware_interface.xacro"/>
     <xacro:include filename="link_macros.xacro"/>
 </robot>
