Commit message: adding urdf

File: src/prototype/urdf/robot_core.xacro (robot description, xacro)
@@ -1,19 +1,114 @@
 <?xml version="1.0"?>
 <robot xmlns:xacro="http://www.ros.org/wiki/xacro">
-    <xacro:include filename="inertial_macros.xacro"/>
-    <material name="white">
-        <color rgba="1 1 1 1" />
-    </material>
-    <material name="orange">
-        <color rgba="1 0.3 0.1 1"/>
-    </material>
-    <material name="blue">
-        <color rgba="0.2 0.2 1 1"/>
-    </material>
-    <material name="black">
-        <color rgba="0 0 0 1"/>
-    </material>
-    <material name="red">
-        <color rgba="1 0 0 1"/>
-    </material>
+    <xacro:property name="body_length_1" value="8.0"/>
+    <xacro:property name="body_width_1" value="6.0"/>
+    <xacro:property name="body_height_1" value="1.5"/>
+    <xacro:property name="body_length_2" value="8.0"/>
+    <xacro:property name="body_width_2" value="6.0"/>
+    <xacro:property name="body_height_2" value="1.0"/>
+    <link name="base_link"></link>
+    <joint name="base_joint" type="fixed">
+        <parent link="base_link"/>
+        <child link="base_footprint"/>
+        <origin xyz="0.0 0.0 0.0" rpy="0 0 0"/>
+      </joint>
+    <link name="base_footprint">
+    </link>
+    <joint name="chassis_1_joint" type="fixed">
+        <parent link="base_link"/>
+        <child link="chassis_1"/>
+        <origin xyz="0.0 0.0 1.2" rpy="0 0 0" />
+    </joint>
+    <link name="chassis_1">
+        <visual>
+            <geometry>
+                <box size="${body_length_1} ${body_width_1} ${body_height_1} "/>
+            </geometry>
+            <material name="chassis_1_mat_silver">
+                <color rgba="0.75 0.75 0.75 1.0"/>
+            </material>
+        </visual>
+    </link>
+    <joint name="sup_rod_1" type="fixed">
+        <parent link="chassis_1"/>
+        <child link="sup_rod_1"/>
+        <origin xyz="-3.5 2.5 1.15" rpy="0 0 0"/>
+    </joint>
+    <link name="sup_rod_1">
+        <visual>
+            <geometry>
+                <box size="0.2 0.2 0.8"/>
+            </geometry>
+            <material name="sup_ros_2_red">
+                <color rgba="0.8 0.8 0.8"/>
+            </material>
+        </visual>
+    </link>
+    <joint name="sup_rod_2_joint" type="fixed">
+        <parent link="chassis_1"/>
+        <child link="sup_rod_2"/>
+        <origin xyz="3.5 -2.5 1.15" rpy="0 0 0"/>
+    </joint>
+    <link name="sup_rod_2">
+        <visual>
+            <geometry>
+                <box size="0.2 0.2 0.8"/>
+            </geometry>
+            <material name="sup_ros_2_red">
+                <color rgba="0.8 0.8 0.8"/>
+            </material>
+        </visual>
+    </link>
+    <joint name="sup_rod_3_joint" type="fixed">
+        <parent link="chassis_1"/>
+        <child link="sup_rod_3"/>
+        <origin xyz="-3.5 -2.5 1.15" rpy="0 0 0"/>
+    </joint>
+    <link name="sup_rod_3">
+        <visual>
+            <geometry>
+                <box size="0.2 0.2 0.8"/>
+            </geometry>
+            <material name="sup_ros_3_red">
+                <color rgba="0.8 0.8 0.8"/>
+            </material>
+        </visual>
+    </link>
+    <joint name="sup_rod_4_joint" type="fixed">
+        <parent link="chassis_1"/>
+        <child link="sup_rod_4"/>
+        <origin xyz="3.5 2.5 1.15" rpy="0 0 0"/>
+    </joint>
+    <link name="sup_rod_4">
+        <visual>
+            <geometry>
+                <box size="0.2 0.2 0.8"/>
+            </geometry>
+            <material name="sup_ros_4_red">
+                <color rgba="0.8 0.8 0.8"/>
+            </material>
+        </visual>
+    </link>
+    <joint name="chassis_2_joint" type="fixed">
+        <parent link="chassis_1"/>
+        <child link="chassis_2"/>
+        <origin xyz="0.0 0.0 2.05" rpy="0.0 0.0 0.0"/>
+    </joint>
+    <link name="chassis_2">
+        <visual>
+            <geometry>
+                <box size="${body_length_2} ${body_width_2} ${body_height_2}"/>
+                <material name="chassis_2_mat_silver">
+                    <color rgba="0.8 0.8 0.8 1.0"/>
+                </material>
+            </geometry>
+        </visual>
+    </link>
+    <joint name="imu_joint" type="fixed">
+        <parent link="chassis_1"/>
+        <child link="imu_link"/>
+        <axis xyz="0.0 0.0 1.0"/>
+        <origin xyz="0.0 0.0 1.00" rpy="0.0 0.0 0.0"/>
+    </joint>
+    <link name="imu_link"></link>
 </robot>

File: src/prototype/urdf/sattava_main.xacro (robot description, xacro)
@@ -1,4 +1,8 @@
 <?xml version="1.0"?>
 <robot xmlns:xacro="http://www.ros.org/wiki/xacro"  name="robot">
-    <xacro:inlcude filename="robot_core.xacro"/>
+    <xacro:include filename="robot_core.xacro"/>
+    <xacro:include filename="camera.xacro"/>
+    <xacro:include filename="lidar.xacro"/>
+    <xacro:include filename="joint_macros.xacro"/>
+    <xacro:include filename="wheel.xacro"/>
 </robot>

Commit message: adding

File: src/prototype/urdf/robot_core.xacro (robot description, xacro)
@@ -112,3 +112,61 @@
     </joint>
     <link name="imu_link"></link>
+    <ros2_control name="PrototypeMotor" type="system">
+        <hardware>
+          <plugin>diffdrive_arduino/DiffDriveArduinoHardware</plugin>
+          <plugin>motor_control/MotorControl</plugin>
+          <param name="back_left_wheel_name">back_left_wheel_joint</param>
+          <param name="back_right_wheel_name">back_right_wheel_joint</param>
+          <param name="loop_rate">30</param>
+          <param name="device">/dev/serial/by-id/usb-Arduino__www.arduino.cc__0043_44236313735351F0A2C1-if00</param>
+          <param name="baud_rate">115200</param>
+          <param name="timeout">1000</param>
+          <param name="enc_counts_per_rev">5606</param>
+        </hardware>
+        <joint name="back_right_wheel_joint">
+          <command_interface name="velocity">
+            <param name="min">0.0</param>
+            <param name="max">2.0</param>
+          </command_interface>
+          <state_interface name="position" />
+          <state_interface name="velocity" />
+        </joint>
+        <joint name="back_left_wheel_joint">
+          <command_interface name="velocity">
+            <param name="min">0.0</param>
+            <param name="max">2.0</param>
+          </command_interface>
+          <state_interface name="position" />
+          <state_interface name="velocity" />
+        </joint>
+      </ros2_control>
+      <ros2_control name="PrototypeMotor" type="system">
+        <hardware>
+          <plugin>diffdrive_arduino/DiffDriveArduinoHardware</plugin>
+          <plugin>motor_control/MotorControl</plugin>
+          <param name="front_left_wheel_name">back_left_wheel_joint</param>
+          <param name="front_right_wheel_name">back_right_wheel_joint</param>
+          <param name="loop_rate">30</param>
+          <param name="device">/dev/serial/by-id/usb-Arduino__www.arduino.cc__0043_850363032323517102E0-if00</param>
+          <param name="baud_rate">115200</param>
+          <param name="timeout">1000</param>
+          <param name="enc_counts_per_rev">5606</param>
+        </hardware>
+        <joint name="front_right_wheel_joint">
+          <command_interface name="velocity">
+            <param name="min">0.0</param>
+            <param name="max">2.0</param>
+          </command_interface>
+          <state_interface name="position" />
+          <state_interface name="velocity" />
+        </joint>
+        <joint name="front_left_wheel_joint">
+          <command_interface name="velocity">
+            <param name="min">0.0</param>
+            <param name="max">2.0</param>
+          </command_interface>
+          <state_interface name="position" />
+          <state_interface name="velocity" />
+        </joint>
+      </ros2_control>
 </robot>
