Commit message: urdf update

File: src/prototype/urdf/camera.xacro (robot description, xacro)
@@ -5,14 +5,14 @@
             <origin xyz="0 0 0" rpy="0 0 0"/>
             <geometry>
-                <box size="0.15 0.3 0.3"/>
+                <box size="0.015 0.03 0.03"/>
             </geometry>
             <material name="camera_material">
-                <color rgba="0.8 0.8 0.8 1"/>
+                <color rgba="0.8 0.8 0.8 "/>
             </material>
         </visual>
     </link>
     <joint name="camera_joint" type="fixed">
-        <origin xyz="3.8 0 0.65" rpy="0 0 0"/>
-        <parent link="chassis_2"/>
+        <origin xyz="0.38 0 0.09" rpy="0 0 0"/>
+        <parent link="chassis_1"/>
         <child link="camera_link"/>
     </joint>

File: src/prototype/urdf/joint_macros.xacro (robot description, xacro)
@@ -1,6 +1,6 @@
 <?xml version="1.0"?>
 <robot xmlns:xacro="http://www.ros.org/wiki/xacro" name="prototype">
-    <xacro:property name="wheel_radius" value="0.5"/>
-    <xacro:property name="wheel_length" value="0.3"/>
+    <xacro:property name="wheel_radius" value="0.05"/>
+    <xacro:property name="wheel_length" value="0.03"/>
    <!--===============xacro for continuous joints=========================-->
     <xacro:macro name="joint_wheel" params="name origin parent child">

File: src/prototype/urdf/lidar.xacro (robot description, xacro)
@@ -4,5 +4,5 @@
         <visual>
             <geometry>
-                <cylinder radius="0.5" length="0.77"/>
+                <cylinder radius="0.05" length="0.077"/>
             </geometry>
             <material name="black">
@@ -10,13 +10,13 @@
             </material>
         </visual>
-        <visual>
+        <!-- <visual>
             <origin xyz="0 0 0"/>
             <geometry>
-                <cylinder radius="0.01" length="0.1"/>
+                <cylinder radius="0.01" length="0.07"/>
             </geometry>
             <material name="black">
                 <color rgba="0 0 0 1"/>
             </material>
-        </visual>
+        </visual>-->
         <collision>
             <origin rpy="0 0 0" xyz="0 0 0"/>
@@ -32,5 +32,5 @@
     </link>
     <joint name="base_laser_joint" type="fixed">
-        <origin xyz="0.0 0.0 0.75" rpy="0.0 0.0 0.0"/>
+        <origin xyz="0.0 0.0 0.075" rpy="0.0 0.0 0.0"/>
         <parent link="chassis_1"/>
         <child link="base_laser"/>

File: src/prototype/urdf/robot_core.xacro (robot description, xacro)
@@ -1,10 +1,10 @@
 <?xml version="1.0"?>
 <robot xmlns:xacro="http://www.ros.org/wiki/xacro">
-    <xacro:property name="body_length_1" value="8.0"/>
-    <xacro:property name="body_width_1" value="6.0"/>
-    <xacro:property name="body_height_1" value="1.5"/>
-    <xacro:property name="body_length_2" value="8.0"/>
-    <xacro:property name="body_width_2" value="6.0"/>
-    <xacro:property name="body_height_2" value="1.0"/>
+    <xacro:property name="body_length_1" value="0.8"/>
+    <xacro:property name="body_width_1" value="0.6"/>
+    <xacro:property name="body_height_1" value="0.15"/>
+    <xacro:property name="body_length_2" value="0.8"/>
+    <xacro:property name="body_width_2" value="0.6"/>
+    <xacro:property name="body_height_2" value="0.1"/>
     <link name="base_link"></link>
     <joint name="base_joint" type="fixed">
@@ -18,5 +18,5 @@
         <parent link="base_link"/>
         <child link="chassis_1"/>
-        <origin xyz="0.0 0.0 1.2" rpy="0 0 0" />
+        <origin xyz="0.0 0.0 0.12" rpy="0 0 0" />
     </joint>
     <link name="chassis_1">
@@ -33,10 +33,10 @@
         <parent link="chassis_1"/>
         <child link="sup_rod_1"/>
-        <origin xyz="-3.5 2.5 1.15" rpy="0 0 0"/>
+        <origin xyz="-0.35 0.25 0.115" rpy="0 0 0"/>
     </joint>
     <link name="sup_rod_1">
         <visual>
             <geometry>
-                <box size="0.2 0.2 0.8"/>
+                <box size="0.02 0.02 0.08"/>
             </geometry>
             <material name="sup_ros_2_red">
@@ -48,10 +48,10 @@
         <parent link="chassis_1"/>
         <child link="sup_rod_2"/>
-        <origin xyz="3.5 -2.5 1.15" rpy="0 0 0"/>
+        <origin xyz="0.35 -0.25 0.115" rpy="0 0 0"/>
     </joint>
     <link name="sup_rod_2">
         <visual>
             <geometry>
-                <box size="0.2 0.2 0.8"/>
+                <box size="0.02 0.02 0.08"/>
             </geometry>
             <material name="sup_ros_2_red">
@@ -63,10 +63,10 @@
         <parent link="chassis_1"/>
         <child link="sup_rod_3"/>
-        <origin xyz="-3.5 -2.5 1.15" rpy="0 0 0"/>
+        <origin xyz="-0.35 -0.25 0.115" rpy="0 0 0"/>
     </joint>
     <link name="sup_rod_3">
         <visual>
             <geometry>
-                <box size="0.2 0.2 0.8"/>
+                <box size="0.02 0.02 0.08"/>
             </geometry>
             <material name="sup_ros_3_red">
@@ -78,10 +78,10 @@
         <parent link="chassis_1"/>
         <child link="sup_rod_4"/>
-        <origin xyz="3.5 2.5 1.15" rpy="0 0 0"/>
+        <origin xyz="0.35 0.25 0.115" rpy="0 0 0"/>
     </joint>
     <link name="sup_rod_4">
         <visual>
             <geometry>
-                <box size="0.2 0.2 0.8"/>
+                <box size="0.02 0.02 0.08"/>
             </geometry>
             <material name="sup_ros_4_red">
@@ -93,5 +93,5 @@
         <parent link="chassis_1"/>
         <child link="chassis_2"/>
-        <origin xyz="0.0 0.0 2.05" rpy="0.0 0.0 0.0"/>
+        <origin xyz="0.0 0.0 0.205" rpy="0.0 0.0 0.0"/>
     </joint>
     <link name="chassis_2">
@@ -108,6 +108,6 @@
         <parent link="chassis_1"/>
         <child link="imu_link"/>
-        <axis xyz="0.0 0.0 1.0"/>
-        <origin xyz="0.0 0.0 1.00" rpy="0.0 0.0 0.0"/>
+        <axis xyz="0.0 0.0 0.10"/>
+        <origin xyz="0.0 0.0 0.100" rpy="0.0 0.0 0.0"/>
     </joint>
     <link name="imu_link"></link>

File: src/prototype/urdf/wheel.xacro (robot description, xacro)
@@ -30,14 +30,14 @@
    </xacro:macro>
    <!-- *********************wheel links and joints***************************************-->
-<xacro:joint_wheel name="back_right_wheel_joint" origin="-3.5 -3.15 -0.75"
+<xacro:joint_wheel name="back_right_wheel_joint" origin="-0.35 -0.315 -0.075"
 parent="chassis_1" child="back_right_wheel"/>
 <xacro:wheel  wheel_name="back_right_wheel"/>
-<xacro:joint_wheel name="back_left_wheel_joint" origin="-3.5 3.15 -0.75"
+<xacro:joint_wheel name="back_left_wheel_joint" origin="-0.35 0.315 -0.075"
 parent="chassis_1" child="back_left_wheel"/>
 <xacro:wheel  wheel_name="back_left_wheel"/>
-<xacro:joint_wheel name="front_right_wheel_joint" origin="3.5 -3.15 -0.75"
+<xacro:joint_wheel name="front_right_wheel_joint" origin="0.35 -0.315 -0.075"
 parent="chassis_1" child="front_right_wheel"/>
 <xacro:wheel  wheel_name="front_right_wheel"/>
-<xacro:joint_wheel name="front_left_wheel_joint" origin="3.5 3.15 -0.75"
+<xacro:joint_wheel name="front_left_wheel_joint" origin="0.35 0.315 -0.075"
 parent="chassis_1" child="front_left_wheel"/>
 <xacro:wheel  wheel_name="front_left_wheel"/>
