Commit message: updating motor_control and prototype

File: src/prototype/urdf/hardware_interface.xacro (robot description, xacro)
@@ -4,3 +4,51 @@
 <xacro:include filename="$(find prototype)/urdf/joint_macros.xacro"/>
 <xacro:include filename="$(find prototype)/urdf/link_macros.xacro"/>
+<!-- ======================ROS2_CONTROL=======================-->
+    <ros2_control name="PrototypeMotor" type="system">
+        <hardware>
+          <plugin>motor_control/MotorControl</plugin>
+          <param name="back_left_wheel_name">back_left_wheel_joint</param>
+          <param name="back_right_wheel_name">back_right_wheel_joint</param>
+          <param name="front_left_wheel_name">front_left_wheel_joint</param>
+          <param name="front_right_wheel_name">front_right_wheel_joint</param>
+          <param name="loop_rate">30</param>
+          <param name="front_arduino">/dev/serial/by-path/platform-fd500000.pcie-pci-0000:01:00.0-usb-0:1.1:1.0</param>
+          <param name="back_arduino">/dev/serial/by-path/platform-fd500000.pcie-pci-0000:01:00.0-usb-0:1.1:1.0</param>
+          <param name="baud_rate">115200</param>
+          <param name="timeout">1000</param>
+          <param name="enc_counts_per_rev">2202</param>
+        </hardware>
+        <joint name="back_right_wheel_joint">
+          <command_interface name="velocity">
+            <param name="min">0.0</param>
+            <param name="max">10.0</param>
+          </command_interface>
+          <state_interface name="position" />
+          <state_interface name="velocity" />
+        </joint>
+        <joint name="back_left_wheel_joint">
+          <command_interface name="velocity">
+            <param name="min">0.0</param>
+            <param name="max">10.0</param>
+          </command_interface>
+          <state_interface name="position" />
+          <state_interface name="velocity" />
+        </joint>
+          <joint name="front_right_wheel_joint">
+          <command_interface name="velocity">
+            <param name="min">0.0</param>
+            <param name="max">10.0</param>
+          </command_interface>
+          <state_interface name="position" />
+          <state_interface name="velocity" />
+        </joint>
+        <joint name="front_left_wheel_joint">
+          <command_interface name="velocity">
+            <param name="min">0.0</param>
+            <param name="max">10.0</param>
+          </command_interface>
+          <state_interface name="position" />
+          <state_interface name="velocity" />
+        </joint>
+      </ros2_control>
 </robot>

Commit message: updated

File: src/prototype/urdf/hardware_interface.xacro (robot description, xacro)
@@ -13,6 +13,6 @@
           <param name="front_right_wheel_name">front_right_wheel_joint</param>
           <param name="loop_rate">30</param>
-          <param name="front_arduino">/dev/serial/by-path/platform-fd500000.pcie-pci-0000:01:00.0-usb-0:1.1:1.0</param>
-          <param name="back_arduino">/dev/serial/by-path/platform-fd500000.pcie-pci-0000:01:00.0-usb-0:1.1:1.0</param>
+          <param name="front_arduino">/dev/serial/by-path/pci-0000:00:14.0-usb-0:1:1.0</param>
+          <param name="back_arduino">/dev/serial/by-path/pci-0000:00:14.0-usb-0:3:1.0</param>
           <param name="baud_rate">115200</param>
           <param name="timeout">1000</param>

File: src/prototype/urdf/robot_core.xacro (robot description, xacro)
@@ -112,61 +112,3 @@
     </joint>
     <link name="imu_link"></link>
-    <ros2_control name="PrototypeMotor" type="system">
-        <hardware>
-          <plugin>diffdrive_arduino/DiffDriveArduinoHardware</plugin>
-          <plugin>motor_control/MotorControl</plugin>
-          <param name="back_left_wheel_name">back_left_wheel_joint</param>
-          <param name="back_right_wheel_name">back_right_wheel_joint</param>
-          <param name="loop_rate">30</param>
-          <param name="device">/dev/serial/by-id/usb-Arduino__www.arduino.cc__0043_44236313735351F0A2C1-if00</param>
-          <param name="baud_rate">115200</param>
-          <param name="timeout">1000</param>
-          <param name="enc_counts_per_rev">5606</param>
-        </hardware>
-        <joint name="back_right_wheel_joint">
-          <command_interface name="velocity">
-            <param name="min">0.0</param>
-            <param name="max">2.0</param>
-          </command_interface>
-          <state_interface name="position" />
-          <state_interface name="velocity" />
-        </joint>
-        <joint name="back_left_wheel_joint">
-          <command_interface name="velocity">
-            <param name="min">0.0</param>
-            <param name="max">2.0</param>
-          </command_interface>
-          <state_interface name="position" />
-          <state_interface name="velocity" />
-        </joint>
-      </ros2_control>
-      <ros2_control name="PrototypeMotor" type="system">
-        <hardware>
-          <plugin>diffdrive_arduino/DiffDriveArduinoHardware</plugin>
-          <plugin>motor_control/MotorControl</plugin>
-          <param name="front_left_wheel_name">back_left_wheel_joint</param>
-          <param name="front_right_wheel_name">back_right_wheel_joint</param>
-          <param name="loop_rate">30</param>
-          <param name="device">/dev/serial/by-id/usb-Arduino__www.arduino.cc__0043_850363032323517102E0-if00</param>
-          <param name="baud_rate">115200</param>
-          <param name="timeout">1000</param>
-          <param name="enc_counts_per_rev">5606</param>
-        </hardware>
-        <joint name="front_right_wheel_joint">
-          <command_interface name="velocity">
-            <param name="min">0.0</param>
-            <param name="max">2.0</param>
-          </command_interface>
-          <state_interface name="position" />
-          <state_interface name="velocity" />
-        </joint>
-        <joint name="front_left_wheel_joint">
-          <command_interface name="velocity">
-            <param name="min">0.0</param>
-            <param name="max">2.0</param>
-          </command_interface>
-          <state_interface name="position" />
-          <state_interface name="velocity" />
-        </joint>
-      </ros2_control>
 </robot>
